Commit message: updating manifest and flipping fingers

File: models/wsg50_110.xacro (robot description, xacro)
@@ -45,5 +45,5 @@
       <parent link="${prefix}gripper_link"/>
       <child link="${prefix}thumb_link"/>
-      <origin xyz="0 -0.096 0" rpy="3.141 3.141 0"/>
+      <origin xyz="0 -0.096 0" rpy="3.141 0 0"/>
     </joint>
     <joint name="${prefix}index_joint" type="prismatic">
@@ -51,5 +51,5 @@
       <parent link="${prefix}gripper_link"/>
       <child link="${prefix}index_link"/>
-      <origin xyz="0 -0.096 0" rpy="3.141 0 0"/>
+      <origin xyz="0 -0.096 0" rpy="3.141 3.141 0"/>
     </joint>
   </macro>
