Commit message: porting from other package

File: models/example.xacro (robot description, xacro)
@@ -1,6 +1,10 @@
 <?xml version="1.0"?>
 <robot xmlns:xacro="http://www.ros.org/wiki/xacro" name="example_robot">
+  <!-- Create a root link -->
+  <link name="world"/>
+  <!-- Instantiate a wsg50 -->
   <include filename="$(find schunk_wsg50_model)/models/wsg50_110.xacro"/>
-  <wsg50 name="" />
+  <wsg50_110 prefix="" />
+  <!-- Attach the gripper to the root link -->
   <joint name="gripper_joint" type="fixed">
     <parent link="world"/>

File: models/wsg50_110.xacro (robot description, xacro)
@@ -1,8 +1,8 @@
 <?xml version="1.0"?>
 <robot xmlns:xacro="http://www.ros.org/wiki/xacro" name="wsg50">
-  <macro name="wsg50" params="prefix">
+  <macro name="wsg50_110" params="prefix">
     <!-- Materials -->
     <material name="wsg50_Gray">
-      <color rgba="0.3 0.3 0.3 1.0"/>
+      <color rgba="0.7 0.7 0.7 1.0"/>
     </material>
     <material name="wsg50_DarkGray">
@@ -25,5 +25,5 @@
         <origin xyz="0 0 0" rpy="0 0 0"/>
         <geometry>
-          <mesh filename="package://schunk_wsg50_model/meshes/finger.stl"
+          <mesh filename="package://schunk_wsg50_model/meshes/wsg_f.stl"
             scale="0.001 0.001 0.001"/>
         </geometry>
@@ -35,5 +35,5 @@
         <origin xyz="0 0 0" rpy="0 0 0"/>
         <geometry>
-          <mesh filename="package://schunk_wsg50_model/meshes/finger.stl"
+          <mesh filename="package://schunk_wsg50_model/meshes/wsg_f.stl"
             scale="0.001 0.001 0.001"/>
         </geometry>

Commit message: new assets generated

File: models/example.xacro (robot description, xacro)
@@ -4,5 +4,5 @@
   <link name="world"/>
   <!-- Instantiate a wsg50 -->
-  <include filename="$(find schunk_wsg50_model)/models/wsg50_110.xacro"/>
+  <include filename="$(find wsg_description)/models/wsg50_110.xacro"/>
   <wsg50_110 prefix="" />
   <!-- Attach the gripper to the root link -->

File: urdf/wsg50_110.urdf (robot description, URDF)
Before this commit: robot wsg50, 0 links, 0 joints
Links:
- added link wsg50_gripper_link; visual mesh filename=package://wsg_description/meshes/wsg50_110.stl scale=0.001 0.001 0.001
- added link wsg50_index_link; visual mesh filename=package://wsg_description/meshes/wsg_f.stl scale=0.001 0.001 0.001
- added link wsg50_thumb_link; visual mesh filename=package://wsg_description/meshes/wsg_f.stl scale=0.001 0.001 0.001
Joints:
- added joint wsg50_index_joint: type prismatic, parent wsg50_gripper_link, child wsg50_index_link, origin xyz=0 -0.096 0 rpy=3.141 3.141 0, limit lower=0.0 upper=0.055 effort=1000.0 velocity=0.5
- added joint wsg50_thumb_joint: type prismatic, parent wsg50_gripper_link, child wsg50_thumb_link, origin xyz=0 -0.096 0 rpy=3.141 0 0, limit lower=0.0 upper=0.055 effort=1000.0 velocity=0.5

File: urdf/wsg50_110_welded_fingers_stl.urdf (robot description, URDF)
Before this commit: robot wsg50, 0 links, 0 joints
Links:
- added link wsg50_gripper_link; collision mesh filename=package://wsg_description/meshes/wsg50_110.stl scale=0.001 0.001 0.001; visual mesh filename=package://wsg_description/meshes/wsg50_110.stl scale=0.001 0.001 0.001
- added link wsg50_index_link; collision mesh filename=package://wsg_description/meshes/wsg_f.stl scale=0.001 0.001 0.001; visual mesh filename=package://wsg_description/meshes/wsg_f.stl scale=0.001 0.001 0.001
- added link wsg50_thumb_link; collision mesh filename=package://wsg_description/meshes/wsg_f.stl scale=0.001 0.001 0.001; visual mesh filename=package://wsg_description/meshes/wsg_f.stl scale=0.001 0.001 0.001
Joints:
- added joint wsg50_index_joint: type fixed, parent wsg50_gripper_link, child wsg50_index_link, origin xyz=0 -0.096 0 rpy=3.141 3.141 0
- added joint wsg50_thumb_joint: type fixed, parent wsg50_gripper_link, child wsg50_thumb_link, origin xyz=0 -0.096 0 rpy=3.141 0 0
