Commit message: new assets generated

File: urdf/wsg50_110_welded_fingers_box_collision.urdf (robot description, URDF)
Before this commit: robot wsg50, 3 links, 2 joints
Links:
- link wsg50_index_link: geometry collision box size=0.023 0.095150742 0.030000001; visual mesh filename=package://wsg_description/meshes/wsg_f.obj scale=0.001 0.001 0.001
- link wsg50_thumb_link: geometry collision box size=0.023 0.095150742 0.030000001; visual mesh filename=package://wsg_description/meshes/wsg_f.obj scale=0.001 0.001 0.001
